File: PCB/KiCAD/LED-Dimmer.kicad_sch (KiCad schematic)
At the start: 9 parts, among them Q1 BC547, U1 NE555D

Commit message: Add 330ohm resistor
Parts:
- added R1: 330, Resistor_THT:R_Axial_DIN0204_L3.6mm_D1.6mm_P1.90mm_Vertical, symbol Device:R
Connections:
- net at D1.2 (A), D2.2 (A), D3.2 (A): now also R1.2; no longer Q1.3 (E)
- new net: Q1.3 (E), R1.1
Other:
- moved on the sheet: C1, D1, D2, D3

Commit message: Add resistor
Parts:
- R1: footprint Resistor_THT:R_Axial_DIN0204_L3.6mm_D1.6mm_P1.90mm_Vertical -> Resistor_THT:R_Axial_DIN0204_L3.6mm_D1.6mm_P7.62mm_Horizontal
Changed lines of the file:
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@@
 			)
 		)
-		(property "Footprint" "Resistor_THT:R_Axial_DIN0204_L3.6mm_D1.6mm_P1.90mm_Vertical"
+		(property "Footprint" "Resistor_THT:R_Axial_DIN0204_L3.6mm_D1.6mm_P7.62mm_Horizontal"
 			(at 193.802 95.25 90)
 			(effects
